Commit message: added camera to default sim, referenced https://classic.gazebosim.org/tutorials?tut=ros_gzplugins

File: src/uav_gazebo/urdf/uav.xacro (robot description, xacro)
@@ -2,4 +2,5 @@
 <robot name="uav" xmlns:xacro="http://www.ros.org/wiki/xacro">
   <xacro:include filename="$(find uav_gazebo)/urdf/uav.gazebo" />
+  <xacro:property name="camera_link" value="0.05" /> <!-- Size of square 'camera' box -->
   <link name="link">
     <pose>0 0 0.2 0 0 0</pose>
@@ -21,3 +22,30 @@
     </visual>
   </link>
+  <joint name="camera_joint" type="fixed">
+    <axis xyz="0 1 0" />
+    <origin xyz="0 0 -0.04" rpy="0 1.570796 0"/>
+    <parent link="link"/>
+    <child link="camera_link"/>
+  </joint>
+  <!-- Camera -->
+  <link name="camera_link">
+    <collision>
+      <origin xyz="0 0 0" rpy="0 0 0"/>
+      <geometry>
+        <box size="0.01 0.03 0.02"/>
+      </geometry>
+    </collision>
+    <visual>
+      <origin xyz="0 0 0" rpy="0 0 0"/>
+      <geometry>
+        <box size="0.01 0.03 0.02"/>
+      </geometry>
+      <material name="red"/>
+    </visual>
+    <inertial>
+      <mass value="1e-5" />
+      <origin xyz="0 0 0" rpy="0 0 0"/>
+      <inertia ixx="1e-6" ixy="0" ixz="0" iyy="1e-6" iyz="0" izz="1e-6" />
+    </inertial>
+  </link>
 </robot>

Commit message: added grass environmnet, and cam_optical link

File: src/uav_gazebo/urdf/uav.xacro (robot description, xacro)
@@ -49,3 +49,16 @@
     </inertial>
   </link>
+  <!-- generate an optical frame
+      http://www.ros.org/reps/rep-0103.html#suffix-frames
+      so that ros and opencv can operate on the camera frame correctly
+      -->
+  <joint name="camera_optical_joint" type="fixed">
+    <!-- these values have to be these values otherwise the gazebo camera
+        image won't be aligned properly with the frame it is supposedly
+        originating from -->
+    <origin xyz="0 0 0" rpy="${-pi/2} 0 ${-pi/2}"/>
+    <parent link="camera_link"/>
+    <child link="camera_link_optical"/>
+  </joint>
+  <link name="camera_link_optical"></link>
 </robot>

Commit message: uav.gazebo and .xacro cause issues with triangle

File: src/uav_gazebo/urdf/uav.xacro (robot description, xacro)
@@ -2,4 +2,5 @@
 <robot name="uav" xmlns:xacro="http://www.ros.org/wiki/xacro">
   <xacro:include filename="$(find uav_gazebo)/urdf/uav.gazebo" />
+  <xacro:property name="camera_link" value="0.05" /> <!-- Size of square 'camera' box -->
   <link name="link">
     <pose>0 0 0.2 0 0 0</pose>
@@ -21,3 +22,43 @@
     </visual>
   </link>
+  <joint name="camera_joint" type="fixed">
+    <axis xyz="0 1 0" />
+    <origin xyz="0 0 -0.04" rpy="0 1.570796 0"/>
+    <parent link="link"/>
+    <child link="camera_link"/>
+  </joint>
+  <!-- Camera -->
+  <link name="camera_link">
+    <collision>
+      <origin xyz="0 0 0" rpy="0 0 0"/>
+      <geometry>
+        <box size="0.01 0.03 0.02"/>
+      </geometry>
+    </collision>
+    <visual>
+      <origin xyz="0 0 0" rpy="0 0 0"/>
+      <geometry>
+        <box size="0.01 0.03 0.02"/>
+      </geometry>
+      <material name="red"/>
+    </visual>
+    <inertial>
+      <mass value="1e-5" />
+      <origin xyz="0 0 0" rpy="0 0 0"/>
+      <inertia ixx="1e-6" ixy="0" ixz="0" iyy="1e-6" iyz="0" izz="1e-6" />
+    </inertial>
+  </link>
+  <!-- generate an optical frame
+      http://www.ros.org/reps/rep-0103.html#suffix-frames
+      so that ros and opencv can operate on the camera frame correctly
+      -->
+  <joint name="camera_optical_joint" type="fixed">
+    <!-- these values have to be these values otherwise the gazebo camera
+        image won't be aligned properly with the frame it is supposedly
+        originating from -->
+    <origin xyz="0 0 0" rpy="${-pi/2} 0 ${-pi/2}"/>
+    <parent link="camera_link"/>
+    <child link="camera_link_optical"/>
+  </joint>
+  <link name="camera_link_optical"></link>
 </robot>
